File: PCB/MildVR/MildVR.kicad_pcb (KiCad board)
At the start: 2 copper layers, 12 parts, among them J1 WP7B-S040VA1-R6000, J2 WP7B-S040VA1-R6000, J3 ZF5S-15-03-T-WT, J4 ZF5S-15-03-T-WT, J5 GPIO, J6 High Speed Serial, U1 ESP32-S3, U3 BMI270, U4 BMI270

Commit message: Organization and stuff
Parts:
- added C1: 10nF, GRM022C81C103ME01L(10nF):GRM022C81C222KE01L, F.Cu at (61.5, 157.8)
- added C10: 1uF, C0805J105K4RACAUTO(1uF):C0805, F.Cu at (68.3, 158.4)
- added C11: 1uF, C0805J105K4RACAUTO(1uF):C0805, F.Cu at (68.3, 162.8)
- added C12: 1nF, C1005NP01H102J050BA(1nF):CAPC1005X55N, F.Cu at (72.6, 140.1)
- added C13: 1nF, C1005NP01H102J050BA(1nF):CAPC1005X55N, F.Cu at (72.6, 142.1)
- added C14: 1nF, C1005NP01H102J050BA(1nF):CAPC1005X55N, F.Cu at (72.6, 144.0)
- added C15: 1nF, C1005NP01H102J050BA(1nF):CAPC1005X55N, F.Cu at (72.6, 146.0)
- added C16: 1nF, C1005NP01H102J050BA(1nF):CAPC1005X55N, F.Cu at (72.6, 148.0)
- added C17: 1nF, C1005NP01H102J050BA(1nF):CAPC1005X55N, F.Cu at (75.5, 140.1)
- added C18: 1nF, C1005NP01H102J050BA(1nF):CAPC1005X55N, F.Cu at (75.5, 142.1)
- added C19: 1nF, C1005NP01H102J050BA(1nF):CAPC1005X55N, F.Cu at (75.5, 144.0)
- added C2: 100nF, ESR01MZPF4701(4.7k):RESC1005X40N, F.Cu at (65.5, 129.0)
- added C20: 1nF, C1005NP01H102J050BA(1nF):CAPC1005X55N, F.Cu at (75.5, 146.0)
- added C21: 1nF, C1005NP01H102J050BA(1nF):CAPC1005X55N, F.Cu at (75.5, 148.0)
- added C22: 1nF, C1005NP01H102J050BA(1nF):CAPC1005X55N, F.Cu at (78.3, 140.1)
- added C23: 100nF, C1005NP01H102J050BA(1nF):CAPC1005X55N, F.Cu at (78.3, 142.1)
- added C25: 100nF, C1005NP01H102J050BA(1nF):CAPC1005X55N, F.Cu at (78.3, 144.0)
- added C26: 10nF, GRM022C81C103ME01L(10nF):GRM022C81C222KE01L, F.Cu at (30.1, 162.2)
- added C27: 100nF, KAF21BR71H104JM(100nF):CAPC2012X94L, F.Cu at (29.2, 142.3)
- added C28: 100nF, KAF21BR71H104JM(100nF):CAPC2012X94L, F.Cu at (29.2, 145.0)
- added C29: 100nF, KAF21BR71H104JM(100nF):CAPC2012X94L, F.Cu at (29.2, 147.7)
- added C3: 100nF, ESR01MZPF4701(4.7k):RESC1005X40N, F.Cu at (65.5, 131.2)
- added C30: 100nF, KAF21BR71H104JM(100nF):CAPC2012X94L, F.Cu at (29.2, 150.4)
- added C4: 100nF, ESR01MZPF4701(4.7k):RESC1005X40N, F.Cu at (65.5, 133.3)
- added C5: 100nF, KAF21BR71H104JM(100nF):CAPC2012X94L, F.Cu at (61.5, 154.8)
- added C6: 1uF, C0805J105K4RACAUTO(1uF):C0805, F.Cu at (68.3, 141.2)
- added C7: 1uF, C0805J105K4RACAUTO(1uF):C0805, F.Cu at (68.3, 145.6)
- added C8: 1uF, C0805J105K4RACAUTO(1uF):C0805, F.Cu at (68.3, 149.8)
- added C9: 1uF, C0805J105K4RACAUTO(1uF):C0805, F.Cu at (68.3, 154.2)
- added D2: LED, SFH_4556(IR_LED):DIO_SFH_4556, F.Cu at (26.8, 121.8)
- added D3: LED, SFH_4556(IR_LED):DIO_SFH_4556, F.Cu at (33.8, 121.8)
- added D4: LED, SFH_4556(IR_LED):DIO_SFH_4556, F.Cu at (40.9, 121.8)
- added D5: LED, SFH_4556(IR_LED):DIO_SFH_4556, F.Cu at (47.9, 121.8)
- added D6: LED, SFH_4556(IR_LED):DIO_SFH_4556, F.Cu at (55.0, 121.8)
- added D7: LED, SFH_4556(IR_LED):DIO_SFH_4556, F.Cu at (62.0, 121.8)
- added R1: 4.7k, ESR01MZPF4701(4.7k):RESC1005X40N, F.Cu at (65.5, 135.5)
- added R19: 16, ERJU03J160V(16Ohm):RES_ERJU03J160V, F.Cu at (25.6, 142.2)
- added R2: 4.7k, ESR01MZPF4701(4.7k):RESC1005X40N, F.Cu at (65.5, 137.6)
- added R20: 16, ERJU03J160V(16Ohm):RES_ERJU03J160V, F.Cu at (25.6, 144.6)
- added R21: 16, ERJU03J160V(16Ohm):RES_ERJU03J160V, F.Cu at (25.6, 147.1)
- added R22: 16, ERJU03J160V(16Ohm):RES_ERJU03J160V, F.Cu at (25.6, 149.5)
- added R23: 16, ERJU03J160V(16Ohm):RES_ERJU03J160V, F.Cu at (25.6, 152.0)
- added R24: 16, ERJU03J160V(16Ohm):RES_ERJU03J160V, F.Cu at (25.6, 154.4)
- added R25: 4.7k, ESR01MZPF4701(4.7k):RESC1005X40N, F.Cu at (30.1, 157.3)
- added R26: 4.7k, ESR01MZPF4701(4.7k):RESC1005X40N, F.Cu at (30.1, 159.4)
- added R3: 4.7k, ESR01MZPF4701(4.7k):RESC1005X40N, F.Cu at (72.8, 150.0)
- added U2: HMC6301BG46, HMC6301BG46:HMC6301BG46, F.Cu at (58.2, 142.5)
- added U5: BMI270, BMI270:BMI270, F.Cu at (26.2, 158.2)
- added U6: BMI270, BMI270:BMI270, F.Cu at (26.2, 162.3)
- J3: value ZF5S-15-03-T-WT -> CAM1
- J4: value ZF5S-15-03-T-WT -> CAM2
- moved J1 121.8 mm to (45.8, 153.9)
- moved J2 121.8 mm to (45.8, 158.8)
- moved U1 119.3 mm to (27.8, 135.5)
- moved U3 114.4 mm to (62.3, 147.4)
- moved U4 114.4 mm to (62.3, 151.4)
- moved PS1 103.0 mm to (57.0, 147.7)
- moved PS2 103.0 mm to (57.0, 152.3)
- moved PS3 103.0 mm to (57.0, 157.0)
- moved J5 99.0 mm to (51.8, 131.1)
- moved J3 99.0 mm to (47.0, 142.3)
- moved J4 99.0 mm to (47.0, 148.3)
- moved J6 99.0 mm to (51.8, 137.0)
Connections:
- J3 pad 01: unconnected-(J3-Pad01) -> GND
- J3 pad 02: unconnected-(J3-Pad02) -> /CAM0_D0_N
- J3 pad 03: unconnected-(J3-Pad03) -> /CAM0_D0_P
- J3 pad 04: unconnected-(J3-Pad04) -> GND
- J3 pad 05: unconnected-(J3-Pad05) -> /CAM0_D1_N
- J3 pad 06: unconnected-(J3-Pad06) -> /CAM0_D1_P
- J3 pad 07: unconnected-(J3-Pad07) -> GND
- J3 pad 08: unconnected-(J3-Pad08) -> /CAM0_D1_P
- J3 pad 09: unconnected-(J3-Pad09) -> /CAM0_C_P
- J3 pad 10: unconnected-(J3-Pad10) -> GND
- J3 pad 11: unconnected-(J3-Pad11) -> /CAM_GPIO
- J3 pad 13: unconnected-(J3-Pad13) -> /SCL0
- J3 pad 14: unconnected-(J3-Pad14) -> /SDA0
- J3 pad 15: unconnected-(J3-Pad15) -> /3V3
- J4 pad 01: unconnected-(J4-Pad01) -> GND
- J4 pad 02: unconnected-(J4-Pad02) -> /CAM1_D0_N
- J4 pad 03: unconnected-(J4-Pad03) -> /CAM1_D0_P
- J4 pad 04: unconnected-(J4-Pad04) -> GND
- J4 pad 05: unconnected-(J4-Pad05) -> /CAM1_D1_N
- J4 pad 06: unconnected-(J4-Pad06) -> /CAM1_C_P
- J4 pad 07: unconnected-(J4-Pad07) -> GND
- J4 pad 08: unconnected-(J4-Pad08) -> /CAM1_C_P
- J4 pad 09: unconnected-(J4-Pad09) -> /CAM1_C_P
- J4 pad 10: unconnected-(J4-Pad10) -> GND
- J4 pad 11: unconnected-(J4-Pad11) -> /CAM_GPIO
- J4 pad 13: unconnected-(J4-Pad13) -> /SCL1
- J4 pad 14: unconnected-(J4-Pad14) -> /SDA1
- J4 pad 15: unconnected-(J4-Pad15) -> /3V3
- J5 pad 1: unconnected-(J5-Pad1) -> GND
- J5 pad 10: unconnected-(J5-Pad10) -> /TRD0_N
- J5 pad 100: unconnected-(J5-Pad100) -> /nEXTRST
- J5 pad 11: unconnected-(J5-Pad11) -> /TRD2_P
- J5 pad 12: unconnected-(J5-Pad12) -> /TRD0_P
- J5 pad 13: unconnected-(J5-Pad13) -> GND
- J5 pad 14: unconnected-(J5-Pad14) -> GND
- J5 pad 15: unconnected-(J5-Pad15) -> /ETH_LEDY
- J5 pad 16: unconnected-(J5-Pad16) -> /SYNC_IN
- J5 pad 17: unconnected-(J5-Pad17) -> /ETH_LEDG
- J5 pad 18: unconnected-(J5-Pad18) -> /SYNC_OUT
- J5 pad 2: unconnected-(J5-Pad2) -> GND
- J5 pad 20: unconnected-(J5-Pad20) -> /EEPROM_nWP
- J5 pad 21: unconnected-(J5-Pad21) -> Net-(D1-K)
- J5 pad 22: unconnected-(J5-Pad22) -> GND
- J5 pad 23: unconnected-(J5-Pad23) -> GND
- J5 pad 24: unconnected-(J5-Pad24) -> /GPIO26
- J5 pad 25: unconnected-(J5-Pad25) -> /GPIO21
- J5 pad 26: unconnected-(J5-Pad26) -> /GPIO19
- J5 pad 27: unconnected-(J5-Pad27) -> /GPIO20
- J5 pad 28: unconnected-(J5-Pad28) -> /GPIO13
- J5 pad 29: unconnected-(J5-Pad29) -> /GPIO16
- J5 pad 3: unconnected-(J5-Pad3) -> /TRD3_P
- J5 pad 30: unconnected-(J5-Pad30) -> /GPIO6
- J5 pad 31: unconnected-(J5-Pad31) -> /GPIO12
- J5 pad 32: unconnected-(J5-Pad32) -> GND
- J5 pad 33: unconnected-(J5-Pad33) -> GND
- J5 pad 34: unconnected-(J5-Pad34) -> /GPIO5
- J5 pad 35: unconnected-(J5-Pad35) -> /ID_SC
- J5 pad 36: unconnected-(J5-Pad36) -> /ID_SD
- J5 pad 37: unconnected-(J5-Pad37) -> /GPIO7
- J5 pad 38: unconnected-(J5-Pad38) -> /GPIO11
- J5 pad 39: unconnected-(J5-Pad39) -> /GPIO8
- J5 pad 4: unconnected-(J5-Pad4) -> /TRD1_P
- J5 pad 40: unconnected-(J5-Pad40) -> /GPIO9
- J5 pad 41: unconnected-(J5-Pad41) -> /GPIO25
- J5 pad 42: unconnected-(J5-Pad42) -> GND
- J5 pad 43: unconnected-(J5-Pad43) -> GND
- J5 pad 44: unconnected-(J5-Pad44) -> /GPIO10
- J5 pad 45: unconnected-(J5-Pad45) -> /GPIO24
- J5 pad 46: unconnected-(J5-Pad46) -> /GPIO22
- J5 pad 47: unconnected-(J5-Pad47) -> /GPIO23
- J5 pad 48: unconnected-(J5-Pad48) -> /GPIO27
- J5 pad 49: unconnected-(J5-Pad49) -> /GPIO18
- J5 pad 5: unconnected-(J5-Pad5) -> /TRD3_N
- J5 pad 50: unconnected-(J5-Pad50) -> /GPIO17
- J5 pad 51: unconnected-(J5-Pad51) -> /GPIO15
- J5 pad 52: unconnected-(J5-Pad52) -> GND
- J5 pad 53: unconnected-(J5-Pad53) -> GND
- J5 pad 54: unconnected-(J5-Pad54) -> /GPIO4
- J5 pad 55: unconnected-(J5-Pad55) -> /GPIO14
- J5 pad 56: unconnected-(J5-Pad56) -> /CLK
- J5 pad 57: unconnected-(J5-Pad57) -> /SD_CLK
- J5 pad 58: unconnected-(J5-Pad58) -> /SDA
- J5 pad 59: unconnected-(J5-Pad59) -> GND
- J5 pad 6: unconnected-(J5-Pad6) -> /TRD1_N
- J5 pad 60: unconnected-(J5-Pad60) -> GND
- J5 pad 61: unconnected-(J5-Pad61) -> /SD_DAT3
- J5 pad 62: unconnected-(J5-Pad62) -> /SD_CMD
- J5 pad 63: unconnected-(J5-Pad63) -> /SD_DAT0
- J5 pad 65: unconnected-(J5-Pad65) -> GND
- J5 pad 66: unconnected-(J5-Pad66) -> GND
- J5 pad 67: unconnected-(J5-Pad67) -> /SD_DAT1
- J5 pad 69: unconnected-(J5-Pad69) -> /SD_DAT2
- J5 pad 7: unconnected-(J5-Pad7) -> GND
- J5 pad 71: unconnected-(J5-Pad71) -> GND
- J5 pad 74: unconnected-(J5-Pad74) -> GND
- J5 pad 75: unconnected-(J5-Pad75) -> /SD_PWR_ON
- J5 pad 76: unconnected-(J5-Pad76) -> /Reserved
- J5 pad 77: unconnected-(J5-Pad77) -> /5V
- J5 pad 78: unconnected-(J5-Pad78) -> /GPIO_VREF
- J5 pad 79: unconnected-(J5-Pad79) -> /5V
- J5 pad 8: unconnected-(J5-Pad8) -> GND
- J5 pad 80: unconnected-(J5-Pad80) -> /SCL0
- J5 pad 81: unconnected-(J5-Pad81) -> /5V
- J5 pad 82: unconnected-(J5-Pad82) -> /SDA0
- J5 pad 83: unconnected-(J5-Pad83) -> /5V
- J5 pad 84: unconnected-(J5-Pad84) -> /3V3
- J5 pad 85: unconnected-(J5-Pad85) -> /5V
- J5 pad 86: unconnected-(J5-Pad86) -> /3V3
- J5 pad 87: unconnected-(J5-Pad87) -> /5V
- J5 pad 88: unconnected-(J5-Pad88) -> /1V8
- J5 pad 9: unconnected-(J5-Pad9) -> /TRD2_N
- J5 pad 90: unconnected-(J5-Pad90) -> /1V8
- J5 pad 91: unconnected-(J5-Pad91) -> /nRPIBOOT
- J5 pad 92: unconnected-(J5-Pad92) -> /RUN_PG
- J5 pad 93: unconnected-(J5-Pad93) -> /nPWR_LED
- J5 pad 94: unconnected-(J5-Pad94) -> /AIN1
- J5 pad 95: unconnected-(J5-Pad95) -> /nPWER_LED
- J5 pad 96: unconnected-(J5-Pad96) -> /AIN0
- J5 pad 97: unconnected-(J5-Pad97) -> /CAM_GPIO
- J5 pad 98: unconnected-(J5-Pad98) -> GND
- J5 pad 99: unconnected-(J5-Pad99) -> /GLOBAL_EN
- J6 pad 1: unconnected-(J6-Pad1) -> /USBOTG_ID
- J6 pad 10: unconnected-(J6-Pad10) -> /PCIE_CLK_P
- J6 pad 100: unconnected-(J6-Pad100) -> /HDMI0_SCL
- J6 pad 11: unconnected-(J6-Pad11) -> /TV_OUT
- J6 pad 12: unconnected-(J6-Pad12) -> /PCIE_CLK_N
- J6 pad 13: P,GND -> GND
- J6 pad 14: P,GND -> GND
- J6 pad 15: unconnected-(J6-Pad15) -> /CAM1_D0_N
- J6 pad 16: unconnected-(J6-Pad16) -> /PCIE_RX_P
- J6 pad 17: unconnected-(J6-Pad17) -> /CAM1_D0_P
- J6 pad 18: unconnected-(J6-Pad18) -> /PCIE_RX_N
- J6 pad 19: P,GND -> GND
- J6 pad 2: unconnected-(J6-Pad2) -> /PCIE_CLK_nREQ
- J6 pad 20: P,GND -> GND
- J6 pad 21: unconnected-(J6-Pad21) -> /CAM1_D1_N
- J6 pad 22: unconnected-(J6-Pad22) -> /PICE_TX_P
- J6 pad 23: unconnected-(J6-Pad23) -> /CAM1_D1_P
- J6 pad 24: unconnected-(J6-Pad24) -> /PCIE_TX_N
- J6 pad 25: P,GND -> GND
- J6 pad 26: P,GND -> GND
- J6 pad 27: unconnected-(J6-Pad27) -> /CAM1_C_N
- J6 pad 28: unconnected-(J6-Pad28) -> /CAM0_D0_N
- J6 pad 29: unconnected-(J6-Pad29) -> /CAM1_C_P
- J6 pad 3: unconnected-(J6-Pad3) -> /USB2_N
- J6 pad 30: unconnected-(J6-Pad30) -> /CAM0_D0_P
- J6 pad 31: unconnected-(J6-Pad31) -> GND
- J6 pad 32: unconnected-(J6-Pad32) -> GND
- J6 pad 33: unconnected-(J6-Pad33) -> /CAM1_D2_N
- J6 pad 34: unconnected-(J6-Pad34) -> /CAM0_D1_N
- J6 pad 35: unconnected-(J6-Pad35) -> /CAM1_D2_P
- J6 pad 36: unconnected-(J6-Pad36) -> /CAM0_D1_P
- J6 pad 37: P,GND -> GND
- J6 pad 38: P,GND -> GND
- J6 pad 39: unconnected-(J6-Pad39) -> /CAM1_D3_N
- J6 pad 40: unconnected-(J6-Pad40) -> /CAM0_C_N
- J6 pad 41: unconnected-(J6-Pad41) -> /CAM1_D3_P
- J6 pad 42: unconnected-(J6-Pad42) -> /CAM0_C_P
- J6 pad 43: unconnected-(J6-Pad43) -> /HDMI1_HOTPLUG
- J6 pad 44: unconnected-(J6-Pad44) -> GND
- J6 pad 45: unconnected-(J6-Pad45) -> /HGMI1_SDA
- J6 pad 46: unconnected-(J6-Pad46) -> /HDMI1_D2_P
- J6 pad 47: unconnected-(J6-Pad47) -> /HDMI1_SCL
- J6 pad 48: unconnected-(J6-Pad48) -> /HDMI1_D2_N
- J6 pad 49: unconnected-(J6-Pad49) -> /HDMI1_CEC
- J6 pad 5: unconnected-(J6-Pad5) -> /USB2_P
- J6 pad 50: unconnected-(J6-Pad50) -> GND
- J6 pad 51: unconnected-(J6-Pad51) -> /HDMI0_CEC
- J6 pad 52: unconnected-(J6-Pad52) -> /HDMI1_D1_P
- J6 pad 53: unconnected-(J6-Pad53) -> /HDMI0_HOTPLUG
- J6 pad 54: unconnected-(J6-Pad54) -> /HDMI1_D1_N
- J6 pad 55: P,GND -> GND
- J6 pad 56: P,GND -> GND
- J6 pad 57: unconnected-(J6-Pad57) -> /DSI0_D0_N
- J6 pad 58: unconnected-(J6-Pad58) -> /HDMI1_D0_P
- J6 pad 59: unconnected-(J6-Pad59) -> /DSI0_D0_P
- J6 pad 60: unconnected-(J6-Pad60) -> /HDMI1_D0_N
- J6 pad 61: P,GND -> GND
- J6 pad 62: P,GND -> GND
- J6 pad 63: unconnected-(J6-Pad63) -> /DSI0_D1_N
- J6 pad 64: unconnected-(J6-Pad64) -> /HDMI1_CK_P
- J6 pad 65: unconnected-(J6-Pad65) -> /DSI_D1_P
- J6 pad 66: unconnected-(J6-Pad66) -> /HDMI1_CK_N
- J6 pad 67: P,GND -> GND
- J6 pad 68: P,GND -> GND
- J6 pad 69: unconnected-(J6-Pad69) -> /DSI0_C_N
- J6 pad 7: P,GND -> GND
- J6 pad 70: unconnected-(J6-Pad70) -> /HDMI0_D2_P
- J6 pad 71: unconnected-(J6-Pad71) -> /DSI0_C_P
- J6 pad 72: unconnected-(J6-Pad72) -> /HDMI0_D2_N
- J6 pad 73: P,GND -> GND
- J6 pad 74: P,GND -> GND
- J6 pad 75: unconnected-(J6-Pad75) -> /DSI1_D0_N
- J6 pad 76: unconnected-(J6-Pad76) -> /HDMI0_D1_P
- J6 pad 77: unconnected-(J6-Pad77) -> /DSI1_D0_P
- J6 pad 78: unconnected-(J6-Pad78) -> /HDMI0_D1_N
- J6 pad 79: unconnected-(J6-Pad79) -> GND
- J6 pad 8: P,GND -> GND
- J6 pad 80: unconnected-(J6-Pad80) -> GND
- J6 pad 81: unconnected-(J6-Pad81) -> /DSI1_D1_N
- J6 pad 82: unconnected-(J6-Pad82) -> /HDMI0_D0_P
- J6 pad 83: unconnected-(J6-Pad83) -> /DSI1_D1_P
- J6 pad 84: unconnected-(J6-Pad84) -> /HDMI0_D0_N
- J6 pad 85: P,GND -> GND
- J6 pad 86: P,GND -> GND
- J6 pad 87: unconnected-(J6-Pad87) -> /DSI1_C_N
- J6 pad 88: unconnected-(J6-Pad88) -> /HDMI0_CK_P
- J6 pad 89: unconnected-(J6-Pad89) -> /DSI1_C_P
- J6 pad 9: unconnected-(J6-Pad9) -> /PCIE_nRST
- J6 pad 90: unconnected-(J6-Pad90) -> /HDMI0_CK_N
- J6 pad 91: unconnected-(J6-Pad91) -> GND
- J6 pad 92: unconnected-(J6-Pad92) -> GND
- J6 pad 93: unconnected-(J6-Pad93) -> /DSI1_D2_N
- J6 pad 94: unconnected-(J6-Pad94) -> /DSI1_D3_N
- J6 pad 95: unconnected-(J6-Pad95) -> /DSI1_D2_P
- J6 pad 96: unconnected-(J6-Pad96) -> /DSI_D3_P
- J6 pad 97: P,GND -> GND
- J6 pad 98: P,GND -> GND
- J6 pad 99: unconnected-(J6-Pad99) -> /HDMI0_SDA
- PS1 pad 1: 3.3V -> /3V3
- PS1 pad 2: P,GND -> GND
- PS1 pad 3: 3.3V -> /3V3
- PS2 pad 1: 3.3V -> /3V3
- PS2 pad 2: P,GND -> GND
- PS2 pad 3: 3.3V -> /3V3
- PS3 pad 1: 3.3V -> /3V3
- PS3 pad 2: P,GND -> GND
- PS3 pad 3: 3.3V -> /3V3
- U1 pad 2: 3.3V -> /Right Controler/3V3
- U1 pad 3: 3.3V -> /Right Controler/3V3
- U1 pad 33: SPICLK -> unconnected-(U1-SPICLK-Pad33)
- U1 pad 43: Net-(U1-GPIO38) -> unconnected-(U1-GPIO38-Pad43)
- U1 pad 5: Net-(R2--) -> unconnected-(U1-GPIO0-Pad5)
- U1 pad 51: Net-(R13-+) -> unconnected-(U1-GPIO45-Pad51)
- U1 pad 52: Net-(R11-+) -> unconnected-(U1-GPIO46-Pad52)
- U1 pad 57: P,GND -> GND1
- U1 pad 6: Net-(R1--) -> unconnected-(U1-GPIO1-Pad6)
- U3 pad 1: 3.3V -> /3V3
- U3 pad 12: 3.3V -> /3V3
- U3 pad 13: Net-(R1--) -> /CLK
- U3 pad 14: Net-(R2--) -> /SDA
- U3 pad 5: 3.3V -> /3V3
- U3 pad 6: P,GND -> GND
- U3 pad 7: P,GND -> GND
- U3 pad 8: 3.3V -> /3V3
- U4 pad 1: P,GND -> GND
- U4 pad 12: 3.3V -> /3V3
- U4 pad 13: Net-(R1--) -> /CLK
- U4 pad 14: Net-(R2--) -> /SDA
- U4 pad 5: 3.3V -> /3V3
- U4 pad 6: P,GND -> GND
- U4 pad 7: P,GND -> GND
- U4 pad 8: 3.3V -> /3V3
