File: PCB/MildVR/MildVR.kicad_sch (KiCad schematic)
At the start: 57 parts, among them J1 WP7B-S040VA1-R6000, J2 WP7B-S040VA1-R6000, J3 CAM1, J4 CAM2, J5 GPIO, J6 High Speed Serial, Q1 BSS138, U2 HMC6301BG46, U3 BMI270, U4 BMI270

Commit message: Replaced HMC6301 with M.2 PCIe Key E
Parts:
- removed C10, C11, C6, C7, C8, C9: 1uF, C0805J105K4RACAUTO(1uF):C0805, symbol PCM_Generic-50:C,IEC
- removed C12, C13, C14, C15, C16, C17, C18, C19, C20, C21, C22: 1nF, C1005NP01H102J050BA(1nF):CAPC1005X55N, symbol PCM_Generic-50:C,IEC
- removed C23, C25: 100nF, C1005NP01H102J050BA(1nF):CAPC1005X55N, symbol PCM_Generic-50:C,IEC
- removed C24: 100pF, symbol PCM_Generic-50:C,IEC
- removed PS1, PS2, PS3: AP7365-WG-7, AP7365-WG-7:AP7365-WG-7, symbol AP7365-WG-7:AP7365-WG-7
- removed Q1: BSS138, BSS138:SOT95P240X111-3N, symbol BSS138:BSS138
- removed R10, R12, R14, R15, R16, R17: 1.2k, symbol PCM_Generic-50:R,IEEE
- removed R11, R13, R9: 2.2k, symbol PCM_Generic-50:R,IEEE
- removed R3: 4.7k, ESR01MZPF4701(4.7k):RESC1005X40N, symbol PCM_Generic-50:R,IEEE
- removed R4, R7: 2k, symbol PCM_Generic-50:R,IEEE
- removed R5: 2.7k, symbol PCM_Generic-50:R,IEEE
- removed R6: 4k, symbol PCM_Generic-50:R,IEEE
- removed R8: 1k, symbol PCM_Generic-50:R,IEEE
- removed U2: HMC6301BG46, HMC6301BG46:HMC6301BG46, symbol HMC6301BG46:HMC6301BG46
- added C31: 22uF, C0805J105K4RACAUTO(1uF):C0805, symbol PCM_Generic-50:C,IEC
- added C32: 10uF, C0805J105K4RACAUTO(1uF):C0805, symbol PCM_Generic-50:C,IEC
- added C33: 100nF, C0805J105K4RACAUTO(1uF):C0805, symbol PCM_Generic-50:C,IEC
- added D10, D8, D9: LED, symbol Device:LED
- added J7: Bus_M.2_Socket_E, (PCIe)MDT420E03001:MDT420E03001, symbol Connector:Bus_M.2_Socket_E
- added R27, R28, R29: 220, symbol PCM_Generic-50:R,IEEE
- added R30, R31: 2.2k, symbol PCM_Generic-50:R,IEEE
- added U2: LM27761DSGR, (Pump)LM27761DSGR:SON50P200X200X80-9N, symbol (Pump)LM27761DSGR:LM27761DSGR
- added Y1: SG-3030CM, Oscillator:Oscillator_SMD_SeikoEpson_SG3030CM, symbol Oscillator:SG-3030CM
- R18: value 1k -> 220
Connections:
- net 3V3: now also C31.1 (+), C32.1 (+), C33.1 (+), J7.2 (3.3V), J7.4 (3.3V), J7.72 (3.3V), J7.74 (3.3V), R27.2 (-), R28.2 (-), R30.1 (+), R31.2 (-), Y1.1 (VIO), Y1.4 (Vcc)
- net 5V: now also J1.32, J1.36
- net CLK: now also J7.60 (I2C_CLK)
- net GND: now also J1.11, J1.12, J1.13, J1.14, J1.15, J1.16, J1.17, J1.18, J1.19, J1.20, J1.25, J1.26, J1.27, J1.28, J1.34, C31.2 (-), C32.2 (-), C33.2 (-), D10.1 (K), J7.1 (GND), J7.18 (GND), J7.33 (GND), J7.38 (VENDOR_DEFINED), J7.39 (GND), J7.40 (VENDOR_DEFINED), J7.45 (GND), J7.51 (GND), J7.57 (GND), J7.63 (GND), J7.69 (GND), J7.7 (GND), J7.75 (GND), Y1.2 (GND)
- net PCIE_CLK_N: now also J7.49 (REFCLKn0)
- net PCIE_CLK_P: now also J7.47 (REFCLKp0)
- net PCIE_CLK_nREQ: now also J7.53 (~{CLKREQ0})
- net PCIE_RX_N: now also J7.43 (PERn0)
- net PCIE_RX_P: now also J7.41 (PERp0)
- net PCIE_nRST: now also J7.52 (~{PERST0})
- net PICE_TX_P: now also J7.35 (PETp0)
- net SDA: now also J7.58 (I2C_DATA)
- net DSI_D1_P renamed DSI0_D1_P
- new net: D10.2 (A), R29.1 (+)
- new net: J7.42 (VENDOR_DEFINED), R29.2 (-)
- new net: J7.54 (~{W_DISABLE2}), R31.1 (+)
- new net: D8.1 (K), J7.6 (~{LED_1})
- new net: D8.2 (A), R27.1 (+)
- new net: J7.50 (SUSCLK), Y1.3 (OUT)
- new net: D9.2 (A), R28.1 (+)
- new net: J7.56 (~{W_DISABLE1}), R30.2 (-)
- new net: D9.1 (K), J7.16 (~{LED_2})
- new net PICE_TX_N: J7.37 (PETn0)
- no-connect marks 10 -> 44
Other:
- moved on the sheet: J1, J2

Commit message: Replace CM4 connectors with CM3588 ones
Parts:
- removed D1: Green, symbol Device:LED
- removed R18: 220, symbol PCM_Generic-50:R,IEEE
- added J8: CON3, DF40C-100DS-0.4V_51:HIROSE_DF40C-100DS-0.4V_51_, symbol DF40C-100DS-0.4V_51:DF40C-100DS-0.4V_51_
- added J9: CON4, DF40C-100DS-0.4V_51:HIROSE_DF40C-100DS-0.4V_51_, symbol DF40C-100DS-0.4V_51:DF40C-100DS-0.4V_51_
- added R3: 100k, symbol PCM_Generic-50:R,IEEE
- J5: value GPIO -> CON1
- J6: value High Speed Serial -> CON2
Connections:
- net AIN1 is gone; now on net GND: J5.94
- net CAM0_C_N is gone; now on net GND: J6.40
- net CAM1_C_N is gone; now on net GND: J6.27
- net CAM1_D2_N is gone; now on net GND: J6.33
- net CAM1_D3_N is gone; now on net GND: J6.39
- net DSI0_C_N is gone; now on net GND: J6.69
- net DSI0_D0_N is gone; now on net GND: J6.57
- net DSI0_D1_N is gone; now on net GND: J6.63
- net DSI1_C_N is gone; now on net GND: J6.87
- net DSI1_D0_N is gone; now on net GND: J6.75
- net DSI1_D1_N is gone; now on net GND: J6.81
- net DSI1_D2_N is gone; now on net GND: J6.93
- net DSI1_D3_N is gone; now on net GND: J6.94
- net GPIO15 is gone; now on net GND: J5.51
- net GPIO22 is gone; now on net GND: J5.46
- net GPIO23 is gone; now on net CSI1_RX_D2P: J5.47
- net GPIO24 is gone; now on net GND: J5.45
- net GPIO26 is gone; now on net GND: J5.24
- net GPIO5 is gone; now on net GND: J5.34
- net GPIO8 is gone; now on net GND: J5.39
- net GPIO9 is gone; now on net GND: J5.40
- net HDMI0_CEC is gone; now on net GND: J6.51
- net HDMI0_CK_P is gone; now on net GND: J6.88
- net HDMI0_D0_P is gone; now on net GND: J6.82
- net HDMI0_D1_P is gone; now on net GND: J6.76
- net HDMI0_D2_P is gone; now on net GND: J6.70
- net HDMI0_SCL is gone; now on net GND: J6.100
- net HDMI0_SDA is gone; now on net GND: J6.99
- net HDMI1_CK_P is gone; now on net GND: J6.64
- net HDMI1_D0_P is gone; now on net GND: J6.58
- net HDMI1_D1_P is gone; now on net GND: J6.52
- net HDMI1_D2_P is gone; now on net GND: J6.46
- net HGMI1_SDA is gone; now on net GND: J6.45
- net Reserved is gone; now on net GND: J5.76
- net SD_DAT0 is gone; now on net GND: J5.63
- net SD_DAT2 is gone; now on net GND: J5.69
- net TRD0_P is gone; now on net GND: J5.12
- net TRD1_N is gone; now on net VDD_12V: J5.6
- net TRD1_P is gone; now on net VDD_12V: J5.4
- net TRD2_N is gone; now on net VDD_12V: J5.9
- net TRD2_P is gone; now on net GND: J5.11
- net TRD3_N is gone; now on net VDD_12V: J5.5
- net TRD3_P is gone; now on net VDD_12V: J5.3
- net nEXTRST is gone; now on net GND: J5.100
- net nRPIBOOT is gone; now on net GND: J5.91
- net 3V3: now also R3.2 (-); no longer J5.84, J5.86
- net 5V: no longer J5.77, J5.79, J5.81, J5.83, J5.85, J5.87
- net CAM0_C_P: no longer J6.42
- net CAM0_D0_N: no longer J6.28
- net CAM0_D0_P: no longer J6.30
- net CAM0_D1_N: no longer J6.34
- net CAM0_D1_P: no longer J6.36
- net CAM1_C_P: no longer J6.29
- net CAM1_D0_N: no longer J6.15
- net CAM1_D0_P: no longer J6.17
- net CAM1_D1_N: no longer J6.21
- net CAM_GPIO: no longer J5.97
- net CLK: no longer J5.56
- net GND: now also J5.57, J5.58, J5.64, J5.70, J5.73, J5.77, J5.82, J5.88, J6.10, J6.15, J6.16, J6.21, J6.22, J6.28, J6.34, J6.9, J8.1, J8.13, J8.14, J8.19, J8.2, J8.20, J8.25, J8.26, J8.31, J8.32, J8.37, J8.38, J8.44, J8.49, J8.50, J8.56, J8.59, J8.62, J8.7, J8.71, J8.8, J8.84, J8.85, J8.94, J9.1, J9.13, J9.14, J9.19, J9.2, J9.20, J9.25, J9.26, J9.31, J9.32, J9.37, J9.38, J9.43, J9.44, J9.49, J9.50, J9.55, J9.61, J9.62, J9.68, J9.7, J9.8, J9.80, J9.83, J9.96; no longer J5.1, J5.14, J5.2, J5.22, J5.23, J5.32, J5.42, J5.43, J5.53, J5.59, J5.60, J5.65, J5.66, J5.7, J5.71, J5.74, J5.8, J5.98, J6.13, J6.14, J6.19, J6.20, J6.25, J6.26, J6.31, J6.32, J6.37, J6.38, J6.44, J6.50, J6.55, J6.56, J6.61, J6.62, J6.67, J6.68, J6.7, J6.73, J6.74, J6.79, J6.8, J6.80, J6.85, J6.86, J6.91, J6.92, J6.97, J6.98
- net SCL0: no longer J5.80
- net SDA: no longer J5.58
- net SDA0: no longer J5.82
- net SD_CLK: now also J9.60; no longer J5.57
- net HPL: now reaches J6.4
- net MIC_IN: now reaches J6.6
- net GPIO2_C0: now reaches J5.21
- net PMIC_EXT_EN_OUT: now reaches J5.19
- net MIPI_CSI0_RX_D0N: now reaches J5.68
- net LED3_25GLAN_25GLED: now reaches J5.72
- net GPIO2_B3: now reaches J5.89
- net 1V8 renamed P25G_MDIP2
- net P25G_MDIP2: no longer J5.88
- net AIN0 renamed P25G_MDIP3
- net CAM1_D1_P renamed MIPI_DPHY0_TX_D3P
- net CAM1_D2_P renamed MIPI_DPHY0_TX_CLKP
- net CAM1_D3_P renamed MIPI_DPHY0_TX_D1P
- net DSI0_C_P renamed TYPEC0_SSRX1P
- net DSI0_D0_P renamed TYPEC0_SSRX2P
- net DSI0_D1_P renamed TYPEC0_SSTX1P
- net DSI1_C_P renamed TYPEC1_SSTX1P
- net DSI1_D0_P renamed TYPEC1_SSTX2P
- net DSI1_D1_P renamed TYPEC1_SSRX2P
- net DSI1_D2_P renamed TYPEC1_SSRX1P
- net DSI_D3_P renamed TYPEC1_OTG_DP
- net EEPROM_nWP renamed UART2_TX_M0_DEBUG
- net ETH_LEDG renamed PWNON_L
- net ETH_LEDY renamed BOOT_SARADC_IN0
- net GLOBAL_EN renamed GPIO2_B7
- net GPIO10 renamed MIPI_CSI0_RX_D3N
- net GPIO11 renamed MIPI_CSI0_RX_CLK1N
- net GPIO12 renamed GPIO4_C6
- net GPIO13 renamed GPIO4_C3
- net GPIO14 renamed CSI1_RX_CLK0N
- net GPIO16 renamed GPIO2_C4
- net GPIO17 renamed MIPI_CSI0_RX_D2N
- net GPIO18 renamed CSI1_RX_D2P
- net GPIO19 renamed GPIO4_C2
- net GPIO20 renamed GPIO2_C3
- net GPIO21 renamed GPIO2_C2/MIPI_CAM2_PDN_L
- net GPIO25 renamed CSI1_RX_D3P
- net GPIO27 renamed MIPI_CSI0_RX_D2P
- net GPIO4 renamed MIPI_CSI0_RX_CLK0P
- net GPIO6 renamed GPIO4_C4/MIPI_CAM1_RESET_L
- net GPIO7 renamed CSI1_RX_CLK1N
- net GPIO_VREF renamed P25G_MDIP0
- net HDMI0_CK_N renamed TYPEC0_OTG_DP
- net HDMI0_D0_N renamed MIPI_DPHY1_TX_D0P
- net HDMI0_D1_N renamed MIPI_DPHY1_TX_D1P
- net HDMI0_D2_N renamed MIPI_DPHY1_TX_CLKP
- net HDMI0_HOTPLUG renamed TYPEC0_SSTX2P
- net HDMI1_CEC renamed MIPI_DPHY0_TX_D0N
- net HDMI1_CK_N renamed MIPI_DPHY1_TX_D2P
- net HDMI1_D0_N renamed MIPI_DPHY1_TX_D3P
- net HDMI1_D1_N renamed MIPI_DPHY1_RX_D0P
- net HDMI1_D2_N renamed MIPI_DPHY1_RX_D1P
- net HDMI1_HOTPLUG renamed MIPI_DPHY0_TX_D1N
- net HDMI1_SCL renamed MIPI_DPHY0_TX_D0P
- net ID_SC renamed CSI1_RX_CLK1P
- net ID_SD renamed MIPI_CSI0_RX_CLK1P
- net PCIE_CLK_N renamed MIPI_DPHY0_RX_D3P
- net MIPI_DPHY0_RX_D3P: no longer J7.49 (REFCLKn0)
- net PCIE_CLK_P renamed PCIE30_PORT0_REFCLKP
- net PCIE30_PORT0_REFCLKP: now also J8.16; no longer J6.10
- net PCIE_CLK_nREQ: no longer names the net of J7.53 (~{CLKREQ0})
- net PCIE_CLK_nREQ: no longer J6.2
- net PCIE_RX_N renamed MIPI_DPHY0_RX_CLKP
- net MIPI_DPHY0_RX_CLKP: no longer J7.43 (PERn0)
- net PCIE_RX_P renamed PCIE30_PORT0_RX1P
- net PCIE30_PORT0_RX1P: now also J8.10; no longer J6.16
- net PCIE_TX_N renamed MIPI_DPHY0_RX_D0P
- net PCIE_nRST renamed GPIO4_B6/PCIE30X4_PERSTn_M1_L
- net GPIO4_B6/PCIE30X4_PERSTn_M1_L: now also J8.69, R3.1 (+); no longer J6.9
- net PICE_TX_N renamed PCIE30_PORT0_TX1N
- net PCIE30_PORT0_TX1N: now also J8.30
- net PICE_TX_P renamed PCIE30_PORT0_TX1P
- net PCIE30_PORT0_TX1P: now also J8.28; no longer J6.22
- net RUN_PG renamed P25G_MDIN2
- net SD_CMD renamed MIPI_CSI0_RX_D1N
- net SD_DAT1 renamed MIPI_CSI1_RX_D0N
- net SD_DAT3 renamed CSI1_RX_D1N
- net SD_PWR_ON renamed GPIO1_B7/MIPI_CAM2_CLKOUT
- net SYNC_IN renamed RESET_L
- net SYNC_OUT renamed VDC_MODE
- net TRD0_N renamed VDD_12V
- net VDD_12V: now also J5.1, J5.2, J5.7, J5.8
- net TV_OUT renamed MIPI_DPHY0_RX_D2P
- net USB2_N renamed HPR
- net USB2_P renamed I2C7_SDA_M0
- net USBOTG_ID renamed RECOVERY
- net nPWER_LED renamed GPIO2_B5
- net nPWR_LED renamed GPIO2_B4
- new net CSI1_RX_CLK0P: J5.53
- new net CSI1_RX_D1P: J5.59
- new net CSI1_RX_D3N: J5.43
- new net GND_AUDIO: J6.2
- new net GPIO0_A4/SDMMC_DET_L: J9.70
- new net GPIO0_B2: J8.47
- new net GPIO0_C4/UART0_RX_M0: J8.70
- new net GPIO0_C5/UART0_TX_M0/PWM4_M0: J8.72
- new net GPIO0_C6/PWM5_M1: J8.74
- new net GPIO0_D3/CC_INT_L: J8.64
- new net GPIO0_D4/PWM3_IR_M0: J8.66
- new net GPIO0_D5: J8.68
- new net GPIO1_A0/UART6_RX_M1: J8.73
- new net GPIO1_A1/UART6_TX_M1: J8.75
- new net GPIO1_A2/I2C4_SDA_M3_TP: J8.77
- new net GPIO1_A3/I2C4_SCL_M3_TP: J8.79
- new net GPIO1_A4: J8.81
- new net GPIO1_A7: J8.83
- new net GPIO1_B0: J8.76
- new net GPIO1_B1/SPI0_MISO_M2: J8.78
- new net GPIO1_B2/SPI0_MOSI_M2/UART4_RX_M2: J8.80
- new net GPIO1_B3/SPI0_CLK_M2/UART4_TX_M2: J8.82
- new net GPIO1_B4/SPI0_CS0_M2/UART7_RX_M2: J8.90
- new net GPIO1_B5/SPI0_CS1_M0/UART7_TX_M2: J8.92
- new net GPIO1_B6/MIPI_CAM1_CLKOUT: J5.71
- new net GPIO1_C0/I2C3_SDA_M0: J8.45
- new net GPIO1_C1/I2C3_SCL_M0: J8.43
- new net GPIO1_C4/HP_DET_L: J6.8
- new net GPIO1_D2/TYPEC5V_PWREN_H: J8.39
- new net GPIO1_D3/PWM1_M1: J8.41
- new net GPIO1_D5/HDMIIRX_DET_L: J8.99
- new net GPIO1_D6/I2C8_SCL_M2: J8.86
- new net GPIO1_D7/I2C8_SDA_M2: J8.88
- new net GPIO2_A6: J5.79
- new net GPIO2_A7: J5.81
- new net GPIO2_B0: J5.83
- new net GPIO2_B1: J5.85
- new net GPIO2_B2: J5.87
- new net GPIO2_B6: J5.97
- new net GPIO2_C1/MIPI_CAM2_RESET_L: J5.23
- new net GPIO3_A0/SPI4_MISO_M1/PWM10_M0: J9.87
- new net GPIO3_A1/SPI4_MOSI_M1: J9.89
- new net GPIO3_A2/SPI4_CLK_M1/UART8_TX_M1: J9.91
- new net GPIO3_A3/SPI4_CS0_M1/UART8_RX_M1: J9.93
- new net GPIO3_A4/SPI4_CS1_M1: J9.95
- new net GPIO3_A5: J9.97
- new net GPIO3_A6/LCD_RST: J9.99
- new net GPIO3_A7: J9.100
- new net GPIO3_B0/PWM9_M0: J9.82
- new net GPIO3_B1/PWM2_M1/LCD_BL: J9.84
- new net GPIO3_B2: J9.86
- new net GPIO3_B3: J9.88
- new net GPIO3_B4: J9.90
- new net GPIO3_B5/UART3_TX_M1/PWM12_M0: J9.92
- new net GPIO3_B6/UART3_RX_M1/PWM13_M0: J9.94
- new net GPIO3_B7: J9.98
- new net GPIO3_C0/TP_INT_L: J8.87
- new net GPIO3_C1/TP_RST_L: J8.89
- new net GPIO3_C2/PWM14_M0: J8.91
- new net GPIO3_C3/PWM15_IR_M0: J8.93
- new net GPIO3_C7/I2C5_SCL_M0_TP: J9.81
- new net GPIO3_D0/I2C5_SDA_M0_TP: J9.79
- new net GPIO3_D5/PWM11_M3/LCD_2_BL: J9.85
- new net GPIO4_A0/TP_2_INT_L: J8.51
- new net GPIO4_A1/TP_2_RST_L: J8.53
- new net GPIO4_A2: J8.55
- new net GPIO4_A3/LCD_2_RST: J8.57
- new net GPIO4_B0/USB_HOST_PWREN_H: J8.61
- new net GPIO4_B3: J8.63
- new net GPIO4_B4/PCIE30X4_CLKREQn_M1_L: J8.65
- new net GPIO4_B5: J8.67
- new net GPIO4_C5/MIPI_CAM1_PDN_L: J5.32
- new net HDMI0_TX0N_PORT: J9.47
- new net HDMI0_TX0P_PORT: J9.45
- new net HDMI0_TX1N_PORT: J9.41
- new net HDMI0_TX1P_PORT: J9.39
- new net HDMI0_TX2N_PORT: J9.35
- new net HDMI0_TX2P_PORT: J9.33
- new net HDMI0_TX3N_PORT: J9.53
- new net HDMI0_TX3P_PORT: J9.51
- new net HDMI0_TX_ON_H: J9.69
- new net HDMI0_TX_SBDN: J9.59
- new net HDMI0_TX_SBDP: J9.57
- new net HDMI1_TX0N_PORT: J9.17
- new net HDMI1_TX0P_PORT: J9.15
- new net HDMI1_TX1N_PORT: J9.11
- new net HDMI1_TX1P_PORT: J9.9
- new net HDMI1_TX2N_PORT: J9.5
- new net HDMI1_TX2P_PORT: J9.3
- new net HDMI1_TX3N_PORT: J9.23
- new net HDMI1_TX3P_PORT: J9.21
- new net HDMI1_TX_ON_H: J9.77
- new net HDMI1_TX_SBDN: J9.29
- new net HDMI1_TX_SBDP: J9.27
- new net HDMIIRX_HPDOUT_H: J9.78
- new net HDMITX0_CEC_M0: J9.67
- new net HDMITX0_HPDIN_M0: J8.95
- new net HDMITX0_SCL_M0: J9.63
- new net HDMITX0_SDA_M0: J9.65
- new net HDMITX1_CEC_M2: J9.75
- new net HDMITX1_HPDIN_M0: J8.97
- new net HDMITX1_SCL_M1: J9.71
- new net HDMITX1_SDA_M1: J9.73
- new net HDMI_RX_CEC: J9.76
- new net HDMI_RX_CLKN_PORT: J9.48
- new net HDMI_RX_CLKP_PORT: J9.46
- new net HDMI_RX_D0N_PORT: J9.42
- new net HDMI_RX_D0P_PORT: J9.40
- new net HDMI_RX_D1N_PORT: J9.36
- new net HDMI_RX_D1P_PORT: J9.34
- new net HDMI_RX_D2N_PORT: J9.30
- new net HDMI_RX_D2P_PORT: J9.28
- new net HDMI_RX_SCL_M1: J9.72
- new net HDMI_RX_SDA_M1: J9.74
- new net I2C6_SCL_M0: J8.96
- new net I2C6_SDA_M0: J8.98
- new net I2C7_SCL_M0: J6.7
- new net LED2_25GLAN_1GLED: J5.74
- new net MIPI_CSI0_RX_CLK0N: J5.56
- new net MIPI_CSI0_RX_D0P: J5.66
- new net MIPI_CSI0_RX_D1P: J5.60
- new net MIPI_CSI0_RX_D3P: J5.42
- new net MIPI_CSI1_RX_D0P: J5.65
- new net MIPI_DPHY0_RX_CLKN: J6.20
- new net MIPI_DPHY0_RX_D0N: J6.26
- new net MIPI_DPHY0_RX_D1N: J6.19
- new net MIPI_DPHY0_RX_D1P: J6.17
- new net MIPI_DPHY0_RX_D2N: J6.13
- new net MIPI_DPHY0_RX_D3N: J6.14
- new net MIPI_DPHY0_TX_CLKN: J6.37
- new net MIPI_DPHY0_TX_D2N: J6.31
- new net MIPI_DPHY0_TX_D2P: J6.29
- new net MIPI_DPHY0_TX_D3N: J6.25
- new net MIPI_DPHY1_RX_CLKN: J6.44
- new net MIPI_DPHY1_RX_CLKP: J6.42
- new net MIPI_DPHY1_RX_D0N: J6.56
- new net MIPI_DPHY1_RX_D1N: J6.50
- new net MIPI_DPHY1_RX_D2N: J6.38
- new net MIPI_DPHY1_RX_D2P: J6.36
- new net MIPI_DPHY1_RX_D3N: J6.32
- new net MIPI_DPHY1_RX_D3P: J6.30
- new net MIPI_DPHY1_TX_CLKN: J6.74
- new net MIPI_DPHY1_TX_D0N: J6.86
- new net MIPI_DPHY1_TX_D1N: J6.80
- new net MIPI_DPHY1_TX_D2N: J6.68
- new net MIPI_DPHY1_TX_D3N: J6.62
- new net P25G_MDIN0: J5.80
- new net P25G_MDIN1: J5.86
- new net P25G_MDIN3: J5.98
- new net P25G_MDIP1: J5.84
- new net PCIE20_1_REFCLKN: J8.17
- new net PCIE20_1_REFCLKP: J8.15
- new net PCIE20_1_RXP/SATA30_1_RXN: J8.11
- new net PCIE20_1_RXP/SATA30_1_RXP: J8.9
- new net PCIE20_1_TXN/SATA30_1_TXN: J8.5
- new net PCIE20_1_TXP/SATA30_1_TXP: J8.3
- new net PCIE20_2_REFCLKN: J8.29
- new net PCIE20_2_REFCLKP: J8.27
- new net PCIE20_2_RXN/SATA30_2_RXN: J8.23
- new net PCIE20_2_RXP/SATA30_2_RXP: J8.21
- new net PCIE20_2_TXN/SATA30_2_TXN: J8.35
- new net PCIE20_2_TXN/SATA30_2_TXP: J8.33
- new net PCIE30_PORT0_REFCLKN: J7.49 (REFCLKn0), J8.18
- new net PCIE30_PORT0_RX0N: J8.6
- new net PCIE30_PORT0_RX0P: J8.4
- new net PCIE30_PORT0_RX1N: J7.43 (PERn0), J8.12
- new net PCIE30_PORT0_TX0N: J8.24
- new net PCIE30_PORT0_TX0P: J8.22
- new net PCIE30_PORT1_REFCLKN: J8.60
- new net PCIE30_PORT1_REFCLKP: J8.58
- new net PCIE30_PORT1_RX2N: J8.36
- new net PCIE30_PORT1_RX2P: J8.34
- new net PCIE30_PORT1_RX3N: J8.42
- new net PCIE30_PORT1_RX3P: J8.40
- new net PCIE30_PORT1_TX2N: J8.48
- new net PCIE30_PORT1_TX2P: J8.46
- new net PCIE30_PORT1_TX3N: J8.54
- new net PCIE30_PORT1_TX3P: J8.52
- new net SARADC_VIN6_HW_ID2: J5.14
- new net SDMMC0_CMD: J9.56
- new net SDMMC0_D0: J9.64
- new net SDMMC0_D1: J9.66
- new net SDMMC0_D2: J9.52
- new net SDMMC0_D3: J9.54
- new net TYPEC0_OTG_DM: J6.92
- new net TYPEC0_SBU1_OUT: J9.4
- new net TYPEC0_SBU2_OUT: J9.6
- new net TYPEC0_SSRX1N: J6.73
- new net TYPEC0_SSRX2N: J6.61
- new net TYPEC0_SSTX1N: J6.67
- new net TYPEC0_SSTX2N: J6.55
- new net TYPEC1_OTG_DM: J6.98
- new net TYPEC1_SBU1: J9.10
- new net TYPEC1_SBU2: J9.12
- new net TYPEC1_SSRX1N: J6.97
- new net TYPEC1_SSRX2N: J6.85
- new net TYPEC1_SSTX1N: J6.91
- new net TYPEC1_SSTX2N: J6.79
- new net UART2_RX_M0_DEBUG: J5.22
- new net USB20_HOST0_DM: J9.24
- new net USB20_HOST0_DP: J9.22
- new net USB20_HOST1_DM: J9.18
- new net USB20_HOST1_DP: J9.16
- new net VBAT_RTC: J8.100
- new net VCC3V3_SD_S0: J9.58
- no-connect marks 44 -> 37
Other:
- moved on the sheet: C31, C32, C33, D10, D8, D9, J1, J2, J3, J4, J6, J7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
